File: KiCad/Esmog_snuffelaar.kicad_pcb (KiCad board)
At the start: 2 copper layers, 135 x 66.5 mm, 277 parts, among them J1 Conn_01x03, J10 AudioJack, J2 Conn_01x03, J3 Conn_01x10_Pin, J4 Conn_01x10_Pin, J5 Conn_01x10_Pin, J6 Conn_01x10_Pin, J7 Conn_01x10_Pin, J9 Conn_Coaxial, P1 USB_C_Plug_USB2.0, Q1 2N7002, Q10 2N7002, Q11 2N7002, Q2 2N7002, Q3 BSR17A, Q4 BC547B, Q5 BC547B, Q6 2N7002, Q7 2N7002, Q8 2N7002, Q9 2N7002, SW1 SW_Push, SW2 SW_Push, SW3 SW_Push, U1 TPS62056DGS, U10 74HC590, U11 4017, U2 TPS62056DGS, U3 LM66100DCK, U4 LM66100DCK, U5 STM32L476RGT6, U6 CP2102N-Axx-xQFN24, U7 TJM4558CDT, U8 74HC590, U9 74HC590, Y1 Crystal_GND24

Commit message: changed some out of stock parts
Parts:
- removed J10: AudioJack, AV-5:Audio_jack
- removed the R18 at (136.6, 34.0)
- added J9: AudioJack3_Dual_Switch, footprints:Audio_jack, F.Cu at (144.5, 82.8)
- added Q1: 2N7002, Package_TO_SOT_SMD:SOT-23, F.Cu at (162.8, 71.0)
- added R11: 75R, Resistor_SMD:R_0603_1608Metric_Pad0.98x0.95mm_HandSolder, F.Cu at (163.8, 74.9)
- BT1: footprint AV-5:BatteryHolder_Keystone_2479_3xAAA -> footprints:BatteryHolder_Keystone_2479_3xAAA
- C20, C22, C23: value 10uF -> C_Polarized; footprint Capacitor_SMD:C_0603_1608Metric_Pad1.08x0.95mm_HandSolder -> Capacitor_SMD:CP_Elec_4x5.4
- J8: renamed from J9; footprint AV-5:CONN-TH_AV-5 -> footprints:CONN-TH_AV-5
- L1, L2: footprint Inductor_SMD:L_0603_1608Metric_Pad1.05x0.95mm_HandSolder -> Inductor_SMD:L_APV_APH0420
- moved D1 9.50 mm to (161.8, 75.0), turned to -90 degrees
- moved R30 6.04 mm to (178.5, 67.0)
- moved U7 5.24 mm to (171.0, 73.0)
- moved C20 4.39 mm to (171.3, 67.2), turned to 0 degrees
- moved R9 4.14 mm to (164.0, 65.8)
- moved R10 4.14 mm to (164.0, 67.8)
- moved R31 3.40 mm to (178.9, 74.6)
- moved R32 3.40 mm to (178.9, 72.6)
- moved R33 3.40 mm to (178.9, 70.6)
- moved SW2 3.04 mm to (148.5, 27.0)
- moved R28 2.96 mm to (205.4, 78.6)
- moved R17 2.96 mm to (148.5, 30.0)
- moved C23 2.78 mm to (186.3, 66.5), turned to 0 degrees
- moved L1 2.05 mm to (153.2, 50.5)
- moved C22 1.55 mm to (206.2, 75.0)
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- renumbered C15 to C10, C13 to C11, C11 to C12, C10 to C13, C16 to C15, C12 to C16, J6 to J3, J3 to J4, J7 to J5, J4 to J6, J5 to J7, Q9 to Q10, Q10 to Q11, Q11 to Q12, Q1 to Q2, Q2 to Q3, Q3 to Q4, Q4 to Q5, Q5 to Q6, Q6 to Q7, Q7 to Q8, Q8 to Q9, R11 to R12, R17 to R13, R20 to R14, R12 to R15, R21 to R16, R13 to R17, R14 to R18, R16 to R20, R15 to R21
Connections:
- C20 pad 1: GND -> +1V5
- C20 pad 2: +1V5 -> GND
- D1 pad 2: VOUT_OPAMP -> Net-(D1-A)
- Q2 pad 3: Net-(Q1-D) -> Net-(D2-DIN)
- R13 pad 2: Net-(Q1-D) -> Net-(D2-DIN)
Routing:
- net Net-(C23-Pad2): track 2.74 -> 81.2 mm, vias 0 -> 3
- net Net-(Q6-C): track 99.1 -> 32.2 mm
- net Net-(Q1-D): track 12.8 -> 0.00 mm
- net +5V: track 105.7 -> 118.5 mm, vias 8 -> 10
- net +1V5: track 88.8 -> 99.4 mm
- net Net-(D2-DIN): track 5.21 -> 15.4 mm
- net Net-(U7-1IN-): track 11.6 -> 16.1 mm
- net /MCU/PC3: track 72.2 -> 68.3 mm
- net ADC1_MCU: track 106.0 -> 109.3 mm
- net BAT_PWR: track 94.3 -> 96.7 mm
- net V-_OPAMP: track 5.91 -> 8.13 mm
- net VOUT_OPAMP: track 6.18 -> 8.32 mm, vias 2 -> 0
- net Net-(Q1-S): track 0.00 -> 2.08 mm
- net Net-(D1-A): track 0.00 -> 2.02 mm
- net Net-(U1-SW): track 2.53 -> 4.31 mm
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Other:
- board text added: "Gijs de Vries E-smog snuffelaar V1.0 22-6-26"
- board text removed: "Gijs de Vries E-smog snuffelaar V1.0 [DATE]"
- board text removed: "sniffing esmog"
